Commit message: Added Custom Gripper

File: robot_description/maciv2.urdf.xacro (robot description, xacro)
@@ -2,4 +2,5 @@
 <robot xmlns:xacro="http://www.ros.org/wiki/xacro" name="maciv2">
     <!-- Robot stuff goes here -->
+    <xacro:include filename="$(find krytn)/robot_description/magni/inertial.xacro" />
     <xacro:include filename="$(find ur_description)/urdf/ur_macro.xacro" />
     <xacro:arg name="ur_type" default="ur5e"/>
@@ -8,3 +9,71 @@
     </xacro:ur_robot>
     <link name="world" />
+    <joint name="gripper_joint" type="fixed">
+        <parent link="ur5_tool0" />
+        <child link="gripper_base_link" />
+        <origin xyz="0 0 0" rpy="0 ${-pi/2} 0" />
+    </joint>
+    <link name="gripper_base_link">
+        <visual>
+            <!--gripper_base-->
+            <!-- <origin rpy="0.0 -0.0 0.0" xyz="0.0 0.0 0.0"/> -->
+            <geometry>
+                <mesh filename="file://$(find maciv2)/robot_description/meshes/Unnamed_gripper_base.dae"/>
+            </geometry>
+        </visual>
+        <collision>
+            <!--gripper_base-->
+            <!-- <origin rpy="0.0 -0.0 0.0" xyz="0.0 0.0 0.0"/> -->
+            <geometry>
+                <mesh filename="file://$(find maciv2)/robot_description/meshes/Unnamed_gripper_base.dae"/>
+            </geometry>
+        </collision>
+        <!-- <inertial>
+            <mass value="0.0"/>
+            <origin rpy="0.0 -0.0 0.0" xyz="0.0 0.0 0.0"/>
+            <inertia ixx="0.0" ixy="0.0" ixz="0.0" iyy="0.0" iyz="0.0" izz="0.0"/>
+        </inertial> -->
+    </link>
+    <link name="finger_link">
+        <visual>
+            <!--finger-->
+            <origin rpy="0.0 -0.0 0.0" xyz="0.0 0.0 0.0"/>
+            <geometry>
+                <mesh filename="file://$(find maciv2)/robot_description/meshes/Unnamed_finger.dae"/>
+            </geometry>
+        </visual>
+        <collision>
+            <!--finger-->
+            <origin rpy="0.0 -0.0 0.0" xyz="0.0 0.0 0.0"/>
+            <geometry>
+                <mesh filename="file://$(find maciv2)/robot_description/meshes/Unnamed_finger.dae"/>
+            </geometry>
+        </collision>
+        <xacro:box_inertial x="0.03" y="0.03" z="0.1" mass="1" />
+    </link>
+    <joint name="finger_joint" type="prismatic">
+        <parent link="gripper_base_link"/>
+        <child link="finger_link"/>
+        <origin rpy="0.0 -0.0 0.0" xyz="0.06 0.0 0.0545"/>
+        <axis xyz="0 0 1"/>
+        <limit effort="1000.0" lower="-0.06" upper="0.0" velocity="10.0"/>
+    </joint>
+    <!-- Configure Control of Joints -->
+    <ros2_control name="maciv2" type="system">
+        <hardware>
+            <plugin>ign_ros2_control/IgnitionSystem</plugin>
+        </hardware>
+        <joint name="finger_joint">
+            <command_interface name="position"/>
+            <state_interface name="position">
+                <param name="initial_value">0.0</param>
+            </state_interface>
+            <state_interface name="velocity"/>
+        </joint>
+    </ros2_control>
+    <gazebo>
+        <plugin filename="ign_ros2_control-system" name="ign_ros2_control::IgnitionROS2ControlPlugin">
+            <parameters>$(find maciv2)/config/ros2_controllers.yaml</parameters>
+        </plugin>
+    </gazebo>
 </robot>
